File: Buddy_Line.kicad_sch (KiCad schematic)
At the start: 18 parts, among them J1 AudioJack3, J2 Conn_01x04_Pin, U3 TPA6110A2DGN

Commit message: New form factor
Parts:
- removed J2: Conn_01x04_Pin, Connector_PinHeader_2.54mm:PinHeader_1x04_P2.54mm_Vertical, symbol Connector:Conn_01x04_Pin
- added C2, C4: 10u, Capacitor_SMD:C_0603_1608Metric, symbol Device:C
- added C3, C5: 0.1u, Capacitor_SMD:C_0603_1608Metric, symbol Device:C
- added J2: AudioJack3, Connector_Audio:Jack_3.5mm_QingPu_WQP-PJ398SM_Vertical_CircularHoles, symbol Connector_Audio:AudioJack3
- added J3: Conn_01x06_Pin, Connector_PinSocket_2.54mm:PinSocket_1x06_P2.54mm_Vertical, symbol Connector:Conn_01x06_Pin
- added R5, R6, R7, R8: 1K, Resistor_SMD:R_0805_2012Metric_Pad1.20x1.40mm_HandSolder, symbol Device:R
- J1: footprint Connector_Audio:Jack_3.5mm_CUI_SJ1-3524N_Horizontal -> Connector_Audio:Jack_3.5mm_QingPu_WQP-PJ398SM_Vertical_CircularHoles
Connections:
- net +3.3V: now also J3.5 (Pin_5), R6.2, R7.2
- net GND: now also C3.2, C5.2, J2.S, J3.6 (Pin_6), R5.1, R8.1; no longer J1.TN
- net DAC_2: now reaches C14.2
- net DAC_2: now also J3.2 (Pin_2)
- net DAC_1: now reaches C13.2
- net DAC_1: now also J3.1 (Pin_1)
- net at RV1.6: now also J1.TN; no longer J1.R
- new net: C2.2, J2.TN
- new net: C4.2, J2.T
- new net ADC_1: C2.1, C3.1, J3.3 (Pin_3), R5.2, R6.1
- new net ADC_2: C4.1, C5.1, J3.4 (Pin_4), R7.1, R8.2
Other:
- moved on the sheet: H1, H2, H3, H4
